File: Breeze-left.kicad_pcb (KiCad board)
At the start: 2 copper layers, 210.6 x 114.9 mm, 102 parts, among them SW1 CHOCXHSPCB-1U, SW10 CHOCXHSPCB-1U, SW11 CHOCXHSPCB-1U, SW12 CHOCXHSPCB-1U, SW13 CHOCXHSPCB-1U, SW14 CHOCXHSPCB-1U, SW15 CHOCXHSPCB-1U, SW16 CHOCXHSPCB-1U, SW17 CHOCXHSPCB-1U, SW18 CHOCXHSPCB-1U, SW19 CHOCXHSPCB-1U, SW2 CHOCXHSPCB-1U, SW20 CHOCXHSPCB-1U, SW21 CHOCXHSPCB-1U, SW22 CHOCXHSPCB-1U, SW23 CHOCXHSPCB-1U, SW24 CHOCXHSPCB-1U, SW3 CHOCXHSPCB-1U, SW4 CHOCXHSPCB-1U, SW5 CHOCXHSPCB-1U, SW6 CHOCXHSPCB-1U, SW7 CHOCXHSPCB-1U, SW8 CHOCXHSPCB-1U, SW9 CHOCXHSPCB-1U

Commit message: Copy right half to left
Parts:
- added R1: 10kΩ, Resistor_SMD:R_0603_1608Metric, B.Cu at (117.9, 152.7)
- D1, D10, D11, D12, D13, D14, D15, D16, D17, D18, D19, D2, D20, D21, D22, D23, D24, D3, D4, D5, D6, D7, D8, D9, DALF1, DAN1, DMC1, DMC2, DMC3, DMC4, DMC5, DMC6, DRT1, DTC1, DTC2, DTC3, DTC4, DUP1: moved to B.Cu
- DOWN1, LEFT1, MC1, MC2, MC3, MC4, MC5, MC6, RIGHT1, SW1, SW10, SW11, SW12, SW13, SW14, SW15, SW16, SW17, SW18, SW19, SW2, SW20, SW21, SW22, SW23, SW24, SW3, SW4, SW5, SW6, SW7, SW8, SW9, TC1, TC2, TC3, TC4, UP1: footprint Breeze:MX_Choc_Hotswap -> Breeze:MX_Choc_Hotswap_1-Sided
- MCU-MAIN1: footprint Breeze:ProMicro -> Breeze:ProMicro_1-Sided
- RSW-MACRO1: footprint Breeze:TACT_SWITCH_TVBP06 -> Button_Switch_SMD:SW_SPST_TL3342; moved to B.Cu
- USB1: footprint Connector_USB:USB_C_Receptacle_HRO_TYPE-C-31-M-12 -> Keebio-Parts:USB-C-12-Pin-MidMount
- moved DTC2 24.5 mm to (147.3, 195.0), turned to 90 degrees
- moved DTC3 24.1 mm to (164.3, 190.5), turned to 90 degrees
- moved DMC4 18.3 mm to (257.5, 139.0), turned to 90 degrees
- moved DMC3 18.1 mm to (293.2, 115.3), turned to 90 degrees
- moved D10 18.1 mm to (192.9, 128.6), turned to 90 degrees
- moved DMC6 18.1 mm to (293.2, 133.9), turned to 90 degrees
- moved D16 18.0 mm to (192.9, 147.6), turned to 90 degrees
- moved D4 17.9 mm to (193.2, 109.8), turned to 90 degrees
- moved D18 17.6 mm to (231.0, 153.6), turned to 90 degrees
- moved D2 17.3 mm to (154.8, 111.3), turned to 90 degrees
- moved D8 17.1 mm to (155.1, 130.7), turned to 90 degrees
- moved D14 17.1 mm to (155.1, 149.7), turned to 90 degrees
- moved DTC4 17.0 mm to (183.4, 190.5), turned to 90 degrees
- moved D12 17.0 mm to (231.0, 134.5), turned to 90 degrees
- moved D6 16.9 mm to (231.3, 115.5), turned to 90 degrees
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Connections:
- MCU-MAIN1 pad 15.1: GND -> SideSelect
Routing:
- net COL8: track 467.0 -> 304.6 mm, vias 12 -> 5
- net COL7: track 419.5 -> 278.3 mm, vias 15 -> 2
- net COL6: track 405.2 -> 268.0 mm, vias 12 -> 2
- net COL3: track 322.1 -> 196.8 mm, vias 11 -> 1
- net COL4: track 304.1 -> 187.1 mm, vias 9 -> 1
- net COL2: track 296.8 -> 183.4 mm, vias 11 -> 3
- net COL1: track 281.9 -> 183.6 mm, vias 11 -> 1
- net COL5: track 321.9 -> 231.4 mm, vias 9 -> 1
- net COL0: track 236.8 -> 167.8 mm, vias 11 -> 1
- net GND: track 383.1 -> 314.0 mm, vias 8 -> 29
- net ROW1: track 272.2 -> 212.4 mm, vias 5 -> 10
- net DATA2: track 17.0 -> 67.8 mm, vias 1 -> 2
- net Net-(DTC3-A): track 60.1 -> 9.41 mm, vias 1 -> 0
- net Net-(D3-A): track 51.9 -> 9.16 mm, vias 1 -> 0
- net Net-(D11-A): track 51.5 -> 9.75 mm, vias 1 -> 0
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- added copper zone on B.Cu, net GND
- added copper zone on F.Cu, net GND
Other:
- outline, holes or cut-outs redrawn
- board text added: "AfternoonLabs.com Breeze Board Rev 1.3 Right Hand Top"
- board text added: "AfternoonLabs.com Gust Macro Board Rev 1.3"
- board text removed: "AfternoonLabs.com Breeze Board Rev1.2 Left Hand Top"
- board text removed: "AfternoonLabs.com Breeze Board Rev1.2 Right Hand Top"
- board text removed: "AfternoonLabs.com Gust Macro Board Rev1.2"
- board text removed: "Snap-Off for Left Hand"

Commit message: Route left hal
Parts:
- removed DALF1, DAN1, DMC1, DMC2, DMC3, DMC4, DMC5, DMC6, DRT1, DUP1: DIODE, Breeze:SOD-123FL
- removed DOWN1, LEFT1, MC1, MC2, MC3, MC4, MC5, MC6, RIGHT1, UP1: CHOCXHSPCB-1U, Breeze:MX_Choc_Hotswap_1-Sided
- removed H1, H16, H17: M3-HOLE, Breeze:M3-HOLE
- removed H10, H11, H12, H13, H14, H15: 2M-HOLE, Breeze:M2-HOLE
- removed MCU-MACRO1: ProMicro-Partial, Breeze:PROMICRO-PARTIAL2
- removed RSW-MACRO1: SW-RST, Button_Switch_SMD:SW_SPST_TL3342
- H18, H19, H2, H3, H4, H5, H6, H7, H8, H9, LGO1, STABL1: moved to B.Cu
- moved USB1 195.6 mm to (303.6, 158.9), turned to 150 degrees
- moved RSW1 181.9 mm to (296.8, 173.2)
- moved R1 163.4 mm to (281.0, 143.8), turned to 90 degrees
- moved MCU-MAIN1 160.6 mm to (286.2, 135.8)
- moved LGO1 160.2 mm to (285.9, 156.7), turned to 180 degrees
- moved STABL1 152.6 mm to (282.1, 187.0), turned to -120 degrees
- moved TC1 152.6 mm to (282.1, 187.0), turned to 60 degrees
- moved DTC1 128.7 mm to (264.9, 190.8)
- moved H9 126.7 mm to (269.2, 179.6), turned to 180 degrees
- moved D19 119.1 mm to (256.9, 173.5)
- moved SW1 119.0 mm to (265.3, 108.2)
- moved SW13 119.0 mm to (265.3, 146.3)
- moved SW19 119.0 mm to (265.3, 165.4)
- moved SW7 119.0 mm to (265.3, 127.2)
- moved D1 117.1 mm to (254.8, 111.0)
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Connections:
- MCU-MAIN1 pad 10: COL6 -> unconnected-(MCU-MAIN1-D7(PE6)-Pad10)
- MCU-MAIN1 pad 11: COL7 -> unconnected-(MCU-MAIN1-D8(PB4)-Pad11)
- MCU-MAIN1 pad 12: COL8 -> unconnected-(MCU-MAIN1-D9(PB5)-Pad12)
- R1 pad 2: GND -> VCC
Routing:
- net COL8: track 304.6 -> 0.00 mm, vias 5 -> 0
- net COL7: track 278.3 -> 0.00 mm, vias 2 -> 0
- net COL6: track 268.0 -> 0.00 mm, vias 2 -> 0
- net GND: track 314.0 -> 81.6 mm, vias 29 -> 7
- net ROW3: track 317.6 -> 163.6 mm, vias 16 -> 7
- net ROW0: track 258.7 -> 149.0 mm, vias 15 -> 7
- net ROW1: track 212.4 -> 136.0 mm, vias 10 -> 6
- net ROW2: track 203.8 -> 150.3 mm, vias 11 -> 7
- net COL0: track 167.8 -> 120.7 mm
- net Net-(MCU-MACRO1-RST): track 43.7 -> 0.00 mm, vias 1 -> 0
- net COL1: track 183.6 -> 157.8 mm
- net COL5: track 231.4 -> 209.8 mm
- net ROW4: track 122.1 -> 103.8 mm, vias 6 -> 2
- net RST: track 53.1 -> 70.5 mm, vias 0 -> 2
- net VCC: track 53.8 -> 69.6 mm
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Other:
- board size 210.6 x 114.9 mm -> 149.6 x 114.9 mm
- board text added: "AfternoonLabs.com Breeze Board Rev 1.3 Left Hand Top"
- board text removed: "AfternoonLabs.com Breeze Board Rev 1.3 Right Hand Top"
- board text removed: "AfternoonLabs.com Gust Macro Board Rev 1.3"
- board text removed: "D0"
- board text removed: "D1"
- board text removed: "D2"
- board text removed: "D20"
- board text removed: "D21"
- board text removed: "D3"
- board text removed: "GND"
- board text removed: "GUST RESET"
- board text removed: "Place Pro-Micro Face Down Here For Gust Macro Pad"
- board text removed: "RAW"
- board text removed: "RST"
- board text removed: "VCC"
